File: christmas-tree.kicad_pcb (KiCad board)
At the start: 2 copper layers, 59 x 53 mm, 11 parts, among them IC1 ATTINY85-P, P1 CONN_2, Q1 PHOTO-TRANSISTOR, SW1 SPST

Commit message: Changes from workstation
Routing:
- added copper zone on B.Cu, net (none)
Changed lines of the file:
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@@
     (last_trace_width 1)
     (trace_clearance 0.254)
-    (zone_clearance 0.508)
+    (zone_clearance 1)
     (zone_45_only no)
     (trace_min 0.254)
@@
   (gr_line (start 67 55.5) (end 75 55.5) (angle 90) (layer Edge.Cuts) (width 0.1))
   (gr_line (start 81.5 41) (end 67 55.5) (angle 90) (layer Edge.Cuts) (width 0.1))
-  (segment (start 82.3 46.5) (end 82.3 45.7) (width 1) (layer B.Cu) (net 1) (status 400000))
-  (segment (start 89.5 74.12) (end 86.81 76.81) (width 1) (layer B.Cu) (net 1) (status 800000))
+  (segment (start 82.3 46.5) (end 82.3 45.7) (width 1) (layer B.Cu) (net 1))
+  (segment (start 89.5 74.12) (end 86.81 76.81) (width 1) (layer B.Cu) (net 1))
   (segment (start 89.5 58.226574) (end 89.5 74.12) (width 1) (layer B.Cu) (net 1))
   (segment (start 85.5 54.226574) (end 89.5 58.226574) (width 1) (layer B.Cu) (net 1))
@@
   (segment (start 91.5 81) (end 91 81) (width 1) (layer B.Cu) (net 1))
   (segment (start 91 81) (end 86.81 76.81) (width 1) (layer B.Cu) (net 1))
-  (segment (start 79.1 46.5) (end 79.1 46.9) (width 1) (layer B.Cu) (net 2) (status C00000))
-  (segment (start 79.69 58.19) (end 82 58.19) (width 1) (layer B.Cu) (net 2) (status 800000))
+  (segment (start 79.1 46.5) (end 79.1 46.9) (width 1) (layer B.Cu) (net 2))
+  (segment (start 79.69 58.19) (end 82 58.19) (width 1) (layer B.Cu) (net 2))
   (segment (start 77 55.5) (end 79.69 58.19) (width 1) (layer B.Cu) (net 2))
   (segment (start 77 49) (end 77 55.5) (width 1) (layer B.Cu) (net 2))
-  (segment (start 79.1 46.9) (end 77 49) (width 1) (layer B.Cu) (net 2) (status 400000))
+  (segment (start 79.1 46.9) (end 77 49) (width 1) (layer B.Cu) (net 2))
   (segment (start 86.81 69.19) (end 86.81 66) (width 1) (layer B.Cu) (net 3))
   (segment (start 86.81 66) (end 87 65.81) (width 1) (layer B.Cu) (net 3))
@@
   (segment (start 81.73 76.81) (end 81.73 80.92) (width 1) (layer B.Cu) (net 7))
   (segment (start 81.73 80.92) (end 81.81 81) (width 1) (layer B.Cu) (net 7))
-  (segment (start 87 58.19) (end 87 57.5) (width 1) (layer B.Cu) (net 8) (status C00000))
-  (segment (start 83.9 47.6) (end 83.9 46.5) (width 1) (layer B.Cu) (net 8) (status 800000))
+  (segment (start 87 58.19) (end 87 57.5) (width 1) (layer B.Cu) (net 8))
+  (segment (start 83.9 47.6) (end 83.9 46.5) (width 1) (layer B.Cu) (net 8))
   (segment (start 82.5 49) (end 83.9 47.6) (width 1) (layer B.Cu) (net 8))
   (segment (start 82.5 53) (end 82.5 49) (width 1) (layer B.Cu) (net 8))
-  (segment (start 87 57.5) (end 82.5 53) (width 1) (layer B.Cu) (net 8) (status 400000))
-  (segment (start 80.7 46.5) (end 80.7 47.8) (width 1) (layer B.Cu) (net 9) (status 400000))
-  (segment (start 84.5 57) (end 84.5 58.19) (width 1) (layer B.Cu) (net 9) (status 800000))
+  (segment (start 87 57.5) (end 82.5 53) (width 1) (layer B.Cu) (net 8))
+  (segment (start 80.7 46.5) (end 80.7 47.8) (width 1) (layer B.Cu) (net 9))
+  (segment (start 84.5 57) (end 84.5 58.19) (width 1) (layer B.Cu) (net 9))
   (segment (start 83.5 56) (end 84.5 57) (width 1) (layer B.Cu) (net 9))
   (segment (start 81 56) (end 83.5 56) (width 1) (layer B.Cu) (net 9))
@@
   (segment (start 72 69.73) (end 74.46 69.73) (width 1) (layer B.Cu) (net 11))
   (segment (start 74.46 69.73) (end 75 69.19) (width 1) (layer B.Cu) (net 11))
+  (zone (net 0) (net_name "") (layer B.Cu) (hatch edge 0.508)
+    (connect_pads (clearance 0.2))
+    (min_thickness 0.254)
+    (fill (arc_segments 16) (thermal_gap 0.508) (thermal_bridge_width 0.508))
+    (polygon
+      (pts
+        (xy 111 87.5) (xy 91 87.5) (xy 91 94) (xy 72 94) (xy 72 87.5)
+        (xy 52 87.5) (xy 67 72.5) (xy 58 72.5) (xy 75 55.5) (xy 67 55.5)
+        (xy 81.5 41) (xy 96 55.5) (xy 88 55.5) (xy 105 72.5) (xy 96 72.5)
+        (xy 111 87.5)
+      )
+    )
+  )
 )

Commit message: Updated PCB to latest version as well
Parts:
- R1: value 10K -> 50K
- SW1: value SPST -> SW_PUSH; footprint SPST_SW -> SW_PUSH_SMALL
- moved D1 125.9 mm to (189.0, 112.0), turned to 90 degrees
- moved R3 103.6 mm to (171.4, 114.3), turned to 0 degrees
- moved R4 100.2 mm to (171.4, 111.8), turned to 0 degrees
- moved R5 96.8 mm to (171.4, 109.2), turned to 0 degrees
- moved C1 93.6 mm to (161.0, 100.0), turned to 180 degrees
- moved SW1 87.6 mm to (173.0, 102.0), turned to 0 degrees
- moved P1 86.1 mm to (161.0, 96.0), turned to 180 degrees
- moved IC1 85.5 mm to (161.0, 108.0), turned to 270 degrees
- moved R2 83.3 mm to (153.7, 100.3)
- moved R1 74.4 mm to (149.9, 100.3), turned to 270 degrees
- moved Q1 72.1 mm to (151.0, 112.0)
Connections:
- IC1 pad 3: N-000008 (its old number) -> N-000004
- IC1 pad 5: N-0000010 -> N-000001
- IC1 pad 6: N-000002 -> N-000003
- IC1 pad 7: N-000003 -> N-000009
- R3 pad 1: N-000003 -> N-000004
- R4 pad 1: N-000002 -> N-000001
- R5 pad 1: N-0000010 -> N-000003
- SW1 pad 2: N-000008 (its old number) -> N-000009
Routing:
- net GND: track 85.6 -> 9.43 mm
- net N-000004: track 0.00 -> 13.3 mm
- net N-000009: track 0.00 -> 12.9 mm
- net N-000008: track 11.3 -> 16.3 mm
- net N-000008 (its old number): track 4.29 -> 0.00 mm
- net N-000002: track 3.48 -> 0.00 mm
- net N-0000010: track 3.46 -> 0.00 mm
- net N-000001: track 0.00 -> 2.85 mm
- net N-000007: track 16.0 -> 13.8 mm
- net N-000006: track 15.7 -> 14.2 mm
- net VCC: track 26.9 -> 28.1 mm
- net N-0000011: track 4.19 -> 3.54 mm
- net N-000003: track 3.49 -> 2.85 mm
- added copper zone on B.Cu, net GND
- removed copper zone on B.Cu, net (none)
Other:
- board outline removed
- board text removed: "2014"
- board text removed: "MakeRiga"
